File: Hardware/C7W1B1V1.0/KiCad/C7W1B1V1.0.sch (KiCad schematic (older format))
At the start: 0 parts

Commit message: początkowy schemat
Changed lines of the file:
@@
 $Descr A4 11693 8268
 encoding utf-8
-Sheet 1 5
+Sheet 1 6
 Title ""
 Date ""
@@
 F1 "Power.sch" 50
 $EndSheet
+$Sheet
+S 1000 2950 1550 1650
+U 672EED17
+F0 "Screen" 50
+F1 "Screen.sch" 50
+$EndSheet
 $EndSCHEMATC
