File: Hardware/C7W1B1V1.0/KiCad/Power.sch (KiCad schematic (older format))
At the start: 0 parts

Commit message: początkowy schemat
Parts:
- added C11, C12, C14, C15, C16, C17, C20, C21, C22: 10u/6.3V/X5R, Capacitor_SMD:C_0402_1005Metric, symbol Device:C
- added C13: 510p/10V/C0G, Capacitor_SMD:C_0402_1005Metric, symbol Device:C
- added C18, C23: 100n/16V/X5R, Capacitor_SMD:C_0402_1005Metric, symbol Device:C
- added D1: PMEG4010CEGWX, Diode_SMD:D_SOD-123, symbol Device:D
- added D2: BZX384B3V3-E3-08, Diode_SMD:D_SOD-323, symbol Device:D
- added F1: 0686F2000-01, Fuse:Fuse_0603_1608Metric, symbol Device:Fuse
- added IC1: USBLC6-2P6, Footprints:USBLC62P6, symbol USBLC6-2P6:USBLC6-2P6
- added IC2: LMR62421XSD_NOPB, Footprints:SON95P300X300X80-7N, symbol LMR62421XSD_NOPB:LMR62421XSD_NOPB
- added IC3: S-8261AAXMD-G2XT2U, Footprints:SOT95P275X135-6N, symbol S-8261AAXMD-G2XT2U:S-8261AAXMD-G2XT2U
- added J3: USB4105GFA120, Footprints:GCT_USB4105GFA120, symbol USB4105GFA120:USB4105GFA120
- added J4: Conn_01x02_Male, TerminalBlock:TerminalBlock_bornier-2_P5.08mm, symbol Connector:Conn_01x02_Male
- added L1: CBC3225T470MR, Inductor_SMD:L_1210_3225Metric, symbol Device:L
- added Q1: PMDPB30XNAX, Footprints:PMDPB30XNAX, symbol PMDPB30XNAX:PMDPB30XNAX
- added R10: 30k/1%/0.063W, Resistor_SMD:R_0402_1005Metric, symbol Device:R
- added R11, R12, R13: 10k/1%/0.063W, Resistor_SMD:R_0402_1005Metric, symbol Device:R
- added R14, R15, R16, R9: 10k/5%/0.063W, Resistor_SMD:R_0402_1005Metric, symbol Device:R
- added R17, R18: 2k2/5%/0.063W, Resistor_SMD:R_0402_1005Metric, symbol Device:R
- added R19: 470/5%/0.063W, Resistor_SMD:R_0402_1005Metric, symbol Device:R
- added R20, R21: 100k/1%/0.063W, Resistor_SMD:R_0402_1005Metric, symbol Device:R
- added U3: STC4054GR, Footprints:SOT95P280X110-5N, symbol STC4054GR:STC4054GR
Connections:
- new net: C13.2, IC2.4 (FB), R10.2, R11.1
- new net: D1.2 (A), IC2.6 (SW), L1.2
- new net: C14.2, C15.2, C16.2, C17.2, C18.2
- new net: R17.1, U3.5 (PROG)
- new net: IC3.1 (DO), Q1.2 (G1)
- new net: Q1.3 (D2_1), Q1.6 (D1__1), Q1.7 (D1__2), Q1.8 (D2_2)
- new net: IC3.3 (CO), Q1.5 (G2)
- new net: IC3.2 (VM), R18.1
- new net: IC3.5 (VDD), R19.1
- new net: J3.A5 (CC1), R14.2
- new net: IC1.3, J3.A6 (DP1), J3.B6 (DP2)
- new net: IC1.1, J3.A7 (DN1), J3.B7 (DN2)
- new net: J3.B5 (CC2), R15.2
- new net +3V3: R16.1
- new net +5V: C13.1, C14.1, C15.1, C16.1, C17.1, C18.1, D1.1 (K), R10.1, R12.1
- new net +BATT: C11.1, C12.1, C23.1, IC2.2 (VIN), J4.2 (Pin_2), L1.1, R19.2, R20.1, U3.3 (BAT)
- new net 5V_EN: IC2.3 (EN), R9.1
- new net 5V_TEST: D2.1 (K), R12.2, R13.1
- new net BATT: R20.2, R21.1
- new net GND: C11.2, C12.2, C20.2, C21.2, C22.2, D2.2 (A), IC1.2, IC2.1 (PGND), IC2.5 (AGND), IC2.7 (EP), J3.A1_B12 (GND), J3.B1_A12 (GND__1), J3.SH1 (SHELL_GND), J3.SH2 (SHELL_GND__1), J3.SH3 (SHELL_GND__2), J3.SH4 (SHELL_GND__3), Q1.4 (S2), R11.2, R13.2, R14.1, R15.1, R17.2, R18.2, R21.2, R9.2, U3.2 (GND)
- new net GND1: C23.2, IC3.6 (VSS), J4.1 (Pin_1), Q1.1 (S1)
- new net USB_D+: IC1.4
- new net USB_D-: IC1.6
- new net VBUS: C20.1, C21.1, C22.1, F1.1, F1.2, IC1.5, J3.A4_B9 (VBUS), J3.B4_A9 (VBUS__1), U3.4 (VCC)
- new net ~CHRG_STATUS: R16.2, U3.1 (CHRG)
- no-connect marks 0 -> 2
