File: Hardware/C7W1B1V1.0/KiCad/Sensor.sch (KiCad schematic (older format))
At the start: 0 parts

Commit message: początkowy schemat
Parts:
- added C10, C8, C9: 100n/16V/X5R, Capacitor_SMD:C_0402_1005Metric, symbol Device:C
- added J2: PMS3003, Connector_PinHeader_2.54mm:PinHeader_2x04_P2.54mm_Vertical, symbol Connector_Generic:Conn_02x04_Counter_Clockwise
- added R4, R5, R6, R7, R8: 10k/5%/0.063W, Resistor_SMD:R_0402_1005Metric, symbol Device:R
- added U2: BME688, Footprints:BME688, symbol BME688:BME688
Connections:
- new net: R5.2, U2.2 (CSB)
- new net: R4.1, U2.5 (SDO)
- new net: J2.2 (Pin_2), R8.2
- new net +3V3: C8.1, C9.1, R5.1, R6.1, R7.1, U2.6 (VDDIO), U2.8 (VDD)
- new net +5V: C10.2, J2.1 (Pin_1), R8.1
- new net GND: C10.1, C8.2, C9.2, J2.8 (Pin_8), R4.2, U2.1 (GND_1), U2.7 (GND_2)
- new net PMS_RST: J2.6 (Pin_6)
- new net PMS_TX: J2.3 (Pin_3)
- new net SCL: R7.2, U2.4 (SCK)
- new net SDA: R6.2, U2.3 (SDI)
- no-connect marks 0 -> 3
