File: Hardware/C7W1B1V1.0/KiCad/Memory.sch (KiCad schematic (older format))
At the start: 0 parts

Commit message: Dodano projekt Cube
Parts:
- added C11, C12: 100n/16V/X5R, Capacitor_SMD:C_0402_1005Metric, symbol Device:C
- added R10, R11, R8, R9: 10k/5%/0.063W, Resistor_SMD:R_0402_1005Metric, symbol Device:R
- added U3: MB85RS512TPNF-G-JNERE1, Footprints:SOIC127P600X175-8N, symbol MB85RS512TPNF-G-JNERE1:MB85RS512TPNF-G-JNERE1
- added U4: W25N512GVEIG, Footprints:SON127P800X600X80-9N-D, symbol W25N512GVEIG:W25N512GVEIG
Connections:
- new net: R8.2, U3.3 (~WP)
- new net: R9.2, U3.7 (~HOLD)
- new net: R10.2, U4.3 (~WP_(IO2))
- new net: R11.2, U4.7 (~HOLD_(IO3))
- new net +3V3: C11.1, C12.1, R10.1, R11.1, R8.1, R9.1, U3.8 (VDD), U4.8 (VCC)
- new net GND: C11.2, C12.2, U3.4 (VSS), U4.4 (GND), U4.9 (EP)
- new net MISO: U3.2 (SO), U4.2 (DO_(IO1))
- new net MOSI: U3.5 (SI), U4.5 (DI_(IO0))
- new net SCK: U3.6 (SCK), U4.6 (CLK)
- new net ~FLASH_CS: U4.1 (~CS)
- new net ~FRAM_CS: U3.1 (~CS)
